File: starbie.kicad_pcb (KiCad board)
At the start: 2 copper layers, 160 x 84.5 mm, 8 parts, among them J1 Conn_01x04_Pin, J2 Conn_01x08_Pin, SW1 SW_Push, SW2 SW_Push, U1 XIAO-ESP32-C3-SMD, U2 DHT11

Commit message: Add files via upload
Parts:
- added G***: LOGO, grapohic:flag, F.Cu at (103.5, 109.5)
- added G***: LOGO, grapohic:H, B.Cu at (204.5, 114.0)
Other:
- board text added: "A PCB by Henry"
